Commit message: Updated m1013.urdf with correct file paths

File: src/m1013/m1013.urdf (robot description, URDF)
Before this commit: robot m1013, 8 links, 7 joints
Links:
- link base_0: geometry collision mesh filename=/pkgs/curobo_doosan/src/m1013/meshes/m1013_collision/MF1013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 scale=0.001 0.001 0.001; visual mesh filename=/pkgs/curobo_doosan/src/m1013/meshes/m1013_white/MF1013_0_0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 scale=0.001 0.001 0.001
- link link1: geometry collision mesh filename=/pkgs/curobo_doosan/src/m1013/meshes/m1013_collision/MF1013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 scale=0.001 0.001 0.001; visual mesh filename=/pkgs/curobo_doosan/src/m1013/meshes/m1013_white/MF1013_1_0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 scale=0.001 0.001 0.001
- link link2: geometry collision mesh filename=/pkgs/curobo_doosan/src/m1013/meshes/m1013_collision/MF1013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 scale=0.001 0.001 0.001; collision mesh filename=/pkgs/curobo_doosan/src/m1013/meshes/m1013_collision/MF1013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 scale=0.001 0.001 0.001
- link link3: geometry collision mesh filename=/pkgs/curobo_doosan/src/m1013/meshes/m1013_collision/MF1013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 scale=0.001 0.001 0.001; visual mesh filename=/pkgs/curobo_doosan/src/m1013/meshes/m1013_white/MF1013_3_0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 scale=0.001 0.001 0.001
- link link4: geometry collision mesh filename=/pkgs/curobo_doosan/src/m1013/meshes/m1013_collision/MF1013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 scale=0.001 0.001 0.001; collision mesh filename=/pkgs/curobo_doosan/src/m1013/meshes/m1013_collision/MF1013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 scale=0.001 0.001 0.001
- link link5: geometry collision mesh filename=/pkgs/curobo_doosan/src/m1013/meshes/m1013_collision/MF1013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 scale=0.001 0.001 0.001; visual mesh filename=/pkgs/curobo_doosan/src/m1013/meshes/m1013_white/MF1013_5_0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 scale=0.001 0.001 0.001
- link link6: geometry collision mesh filename=/pkgs/curobo_doosan/src/m1013/meshes/m1013_collision/MF1013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 scale=0.001 0.001 0.001; visual mesh filename=/pkgs/curobo_doosan/src/m1013/meshes/m1013_white/MF1013_6_0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 scale=0.001 0.001 0.001

Commit message: absolut path to relatif

File: src/m1013/m1013.urdf (robot description, URDF)
Before this commit: robot m1013, 8 links, 7 joints
Links:
- link base_0: geometry collision mesh filename=package://curobo_ros/curobo_doosan/src/m1013/meshes/m1013_c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 scale=0.001 0.001 0.001; visual mesh filename=package://curobo_ros/curobo_doosan/src/m1013/meshes/m1013_w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 scale=0.001 0.001 0.001
- link link1: geometry collision mesh filename=package://curobo_ros/curobo_doosan/src/m1013/meshes/m1013_c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 scale=0.001 0.001 0.001; visual mesh filename=package://curobo_ros/curobo_doosan/src/m1013/meshes/m1013_w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 scale=0.001 0.001 0.001
- link link2: geometry collision mesh filename=package://curobo_ros/curobo_doosan/src/m1013/meshes/m1013_c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 scale=0.001 0.001 0.001; collision mesh filename=package://curobo_ros/curobo_doosan/src/m1013/meshes/m1013_c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 scale=0.001 0.001 0.001
- link link3: geometry collision mesh filename=package://curobo_ros/curobo_doosan/src/m1013/meshes/m1013_c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 scale=0.001 0.001 0.001; visual mesh filename=package://curobo_ros/curobo_doosan/src/m1013/meshes/m1013_w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 scale=0.001 0.001 0.001
- link link4: geometry collision mesh filename=package://curobo_ros/curobo_doosan/src/m1013/meshes/m1013_c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 scale=0.001 0.001 0.001; collision mesh filename=package://curobo_ros/curobo_doosan/src/m1013/meshes/m1013_c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 scale=0.001 0.001 0.001
- link link5: geometry collision mesh filename=package://curobo_ros/curobo_doosan/src/m1013/meshes/m1013_c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 scale=0.001 0.001 0.001; visual mesh filename=package://curobo_ros/curobo_doosan/src/m1013/meshes/m1013_w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 scale=0.001 0.001 0.001
- link link6: geometry collision mesh filename=package://curobo_ros/curobo_doosan/src/m1013/meshes/m1013_c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 scale=0.001 0.001 0.001; visual mesh filename=package://curobo_ros/curobo_doosan/src/m1013/meshes/m1013_w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 scale=0.001 0.001 0.001

Commit message: update accelerations and joint limits

File: src/m1013/m1013.urdf (robot description, URDF)
Before this commit: robot m1013, 8 links, 7 joints
Joints:
- joint joint2: limit lower=-6.2832 upper=6.2832 effort=346 velocity=2.0944 -> lower=-2.0944 upper=2.0944 effort=346 velocity=2.0944
- joint joint3: limit lower=-2.7925 upper=2.7925 effort=163 velocity=3.1416 -> lower=-2.35619 upper=2.35619 effort=163 velocity=3.1416
- joint joint5: limit lower=-6.2832 upper=6.2832 effort=50 velocity=3.927 -> lower=-2.35619 upper=2.35619 effort=50 velocity=3.927

Commit message: joint limit more realiste

File: src/m1013/m1013.urdf (robot description, URDF)
Before this commit: robot m1013, 8 links, 7 joints
Joints:
- joint joint2: limit lower=-2.0944 upper=2.0944 effort=346 velocity=2.0944 -> lower=-6.2832 upper=6.2832 effort=346 velocity=2.0944

Commit message: Convert repository to ROS2 package
- Add ROS2 package structure (package.xml, CMakeLists.txt)
- Create display.launch.py with robot_state_publisher and joint_state_publisher
- Add RViz configuration file for robot visualization
- Update URDF mesh paths to use correct ROS2 package reference
- Add ROS2_USAGE.md with usage instructions in French

File: src/m1013/m1013.urdf (robot description, URDF)
Before this commit: robot m1013, 8 links, 7 joints
Links:
- link base_0: geometry collision mesh filename=package://curobo_doosan/src/m1013/meshes/m1013_collision/MF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 scale=0.001 0.001 0.001; visual mesh filename=package://curobo_doosan/src/m1013/meshes/m1013_white/MF1013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 scale=0.001 0.001 0.001
- link link1: geometry collision mesh filename=package://curobo_doosan/src/m1013/meshes/m1013_collision/MF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 scale=0.001 0.001 0.001; visual mesh filename=package://curobo_doosan/src/m1013/meshes/m1013_white/MF1013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 scale=0.001 0.001 0.001
- link link2: geometry collision mesh filename=package://curobo_doosan/src/m1013/meshes/m1013_collision/MF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 scale=0.001 0.001 0.001; collision mesh filename=package://curobo_doosan/src/m1013/meshes/m1013_collision/MF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 scale=0.001 0.001 0.001
- link link3: geometry collision mesh filename=package://curobo_doosan/src/m1013/meshes/m1013_collision/MF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 scale=0.001 0.001 0.001; visual mesh filename=package://curobo_doosan/src/m1013/meshes/m1013_white/MF1013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 scale=0.001 0.001 0.001
- link link4: geometry collision mesh filename=package://curobo_doosan/src/m1013/meshes/m1013_collision/MF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 scale=0.001 0.001 0.001; collision mesh filename=package://curobo_doosan/src/m1013/meshes/m1013_collision/MF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 scale=0.001 0.001 0.001
- link link5: geometry collision mesh filename=package://curobo_doosan/src/m1013/meshes/m1013_collision/MF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 scale=0.001 0.001 0.001; visual mesh filename=package://curobo_doosan/src/m1013/meshes/m1013_white/MF1013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 scale=0.001 0.001 0.001
- link link6: geometry collision mesh filename=package://curobo_doosan/src/m1013/meshes/m1013_collision/MF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 scale=0.001 0.001 0.001; visual mesh filename=package://curobo_doosan/src/m1013/meshes/m1013_white/MF1013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 scale=0.001 0.001 0.001
