Commit message: refactor URDF and YAML configurations for consistency and clarity

File: src/m1013/m1013.urdf (robot description, URDF)
Before this commit: robot m1013, 8 links, 7 joints
Links:
- removed link base_0
- removed link link1
- removed link link2
- removed link link3
- removed link link4
- removed link link5
- removed link link6
- added link dsr01/link1, mass 7.8; collision mesh filename=package://curobo_ros/curobo_doosan/src/m1013/meshes/m1013_c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 scale=0.001 0.001 0.001; visual mesh filename=package://curobo_ros/curobo_doosan/src/m1013/meshes/m1013_w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 scale=0.001 0.001 0.001
- added link dsr01/link2, mass 10.83; collision mesh filename=package://curobo_ros/curobo_doosan/src/m1013/meshes/m1013_c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 scale=0.001 0.001 0.001; collision mesh filename=package://curobo_ros/curobo_doosan/src/m1013/meshes/m1013_c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 scale=0.001 0.001 0.001
- added link dsr01/link3, mass 3.68; collision mesh filename=package://curobo_ros/curobo_doosan/src/m1013/meshes/m1013_c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 scale=0.001 0.001 0.001; visual mesh filename=package://curobo_ros/curobo_doosan/src/m1013/meshes/m1013_w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 scale=0.001 0.001 0.001
- added link dsr01/link4, mass 3.82; collision mesh filename=package://curobo_ros/curobo_doosan/src/m1013/meshes/m1013_c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 scale=0.001 0.001 0.001; collision mesh filename=package://curobo_ros/curobo_doosan/src/m1013/meshes/m1013_c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 scale=0.001 0.001 0.001
- added link dsr01/link5, mass 2.82; collision mesh filename=package://curobo_ros/curobo_doosan/src/m1013/meshes/m1013_c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 scale=0.001 0.001 0.001; visual mesh filename=package://curobo_ros/curobo_doosan/src/m1013/meshes/m1013_w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 scale=0.001 0.001 0.001
- added link dsr01/link6, mass 1.16; collision mesh filename=package://curobo_ros/curobo_doosan/src/m1013/meshes/m1013_c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 scale=0.001 0.001 0.001; visual mesh filename=package://curobo_ros/curobo_doosan/src/m1013/meshes/m1013_w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 scale=0.001 0.001 0.001
- added link dsr01/world, mass 4.12; collision mesh filename=package://curobo_ros/curobo_doosan/src/m1013/meshes/m1013_c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 scale=0.001 0.001 0.001; visual mesh filename=package://curobo_ros/curobo_doosan/src/m1013/meshes/m1013_w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 scale=0.001 0.001 0.001
Joints:
- joint joint1: child link1 -> dsr01/link1; parent base_0 -> dsr01/world
- joint joint2: child link2 -> dsr01/link2; parent link1 -> dsr01/link1
- joint joint3: child link3 -> dsr01/link3; limit lower=-2.35619 upper=2.35619 effort=163 velocity=3.1416 -> lower=-2.2 upper=2.2 effort=163 velocity=3.1416; parent link2 -> dsr01/link2
- joint joint4: child link4 -> dsr01/link4; parent link3 -> dsr01/link3
- joint joint5: child link5 -> dsr01/link5; parent link4 -> dsr01/link4
- joint joint6: child link6 -> dsr01/link6; parent link5 -> dsr01/link5
- joint world_fixed: child base_0 -> dsr01/world

Commit message: update joint limits and add attached object configuration in YAML

File: src/m1013/m1013.urdf (robot description, URDF)
Before this commit: robot m1013, 8 links, 7 joints
Joints:
- joint joint3: limit lower=-2.2 upper=2.2 effort=163 velocity=3.1416 -> lower=-2.35619 upper=2.35619 effort=163 velocity=3.1416

Commit message: update joint limit 2

File: src/m1013/m1013.urdf (robot description, URDF)
Before this commit: robot m1013, 8 links, 7 joints
Joints:
- joint joint2: limit lower=-6.2832 upper=6.2832 effort=346 velocity=2.0944 -> lower=-2.0944 upper=2.0944 effort=346 velocity=2.0944
- joint joint3: limit lower=-2.35619 upper=2.35619 effort=163 velocity=3.1416 -> lower=-2.61799 upper=2.61799 effort=163 velocity=3.1416
