Commit message: Reorganize package with standard ROS2 structure
- Move meshes from src/m1013/meshes/ to meshes/
- Move URDF from src/m1013/ to urdf/
- Move config files (yml, usd) from src/m1013/ to config/
- Update URDF mesh paths to use package://curobo_doosan/meshes/
- Update launch file to use new URDF path
- Update CMakeLists.txt to install new directories
- Update ROS2_USAGE.md to reflect new structure
- Remove src/ directory

New structure follows ROS2 conventions with separate directories for:
- urdf/: Robot description files
- meshes/: 3D mesh files for visualization and collision
- config/: Configuration and USD files for Isaac Sim
- launch/: Launch files and RViz config

File: urdf/m1013.urdf (robot description, URDF)
Before this commit: robot m1013, 8 links, 7 joints
Links:
- link base_0: geometry collision mesh filename=package://curobo_doosan/meshes/m1013_collision/MF1013_0_0.d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 scale=0.001 0.001 0.001; visual mesh filename=package://curobo_doosan/meshes/m1013_white/MF1013_0_0.dae scale=0.001 0.001 0.001
- link link1: geometry collision mesh filename=package://curobo_doosan/meshes/m1013_collision/MF1013_1_0.d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 scale=0.001 0.001 0.001; visual mesh filename=package://curobo_doosan/meshes/m1013_white/MF1013_1_0.dae scale=0.001 0.001 0.001
- link link2: geometry collision mesh filename=package://curobo_doosan/meshes/m1013_collision/MF1013_2_0.d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 scale=0.001 0.001 0.001; collision mesh filename=package://curobo_doosan/meshes/m1013_collision/MF1013_2_1.d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 scale=0.001 0.001 0.001
- link link3: geometry collision mesh filename=package://curobo_doosan/meshes/m1013_collision/MF1013_3_0.d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 scale=0.001 0.001 0.001; visual mesh filename=package://curobo_doosan/meshes/m1013_white/MF1013_3_0.dae scale=0.001 0.001 0.001
- link link4: geometry collision mesh filename=package://curobo_doosan/meshes/m1013_collision/MF1013_4_0.d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 scale=0.001 0.001 0.001; collision mesh filename=package://curobo_doosan/meshes/m1013_collision/MF1013_4_1.d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 scale=0.001 0.001 0.001
- link link5: geometry collision mesh filename=package://curobo_doosan/meshes/m1013_collision/MF1013_5_0.d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 scale=0.001 0.001 0.001; visual mesh filename=package://curobo_doosan/meshes/m1013_white/MF1013_5_0.dae scale=0.001 0.001 0.001
- link link6: geometry collision mesh filename=package://curobo_doosan/meshes/m1013_collision/MF1013_6_0.d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 scale=0.001 0.001 0.001; visual mesh filename=package://curobo_doosan/meshes/m1013_white/MF1013_6_0.dae scale=0.001 0.001 0.001
